File: schematic/abc-lcd/abc-lcd.kicad_pcb (KiCad board)
At the start: 2 copper layers, 39 parts, among them J1 Screw_Terminal_01x03, J2 USB_A, J3 Screw_Terminal_01x03, J4 Screw_Terminal_01x03, Q1 IRFZ44, SW1 SW_Push, U1 74164, U2 RC1602A, U3 ATmega8A-PU, U4 LM2596S-5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

Commit message: Proper component placement
Parts:
- J1: value Screw_Terminal_01x03 -> 24v-INPUT
- J3: value Screw_Terminal_01x03 -> 24v_OUTPUT
- J4: value Screw_Terminal_01x03 -> ADJ_OUTPUT
- U1, U4, U5: moved to B.Cu
- moved J1 468.1 mm to (-105.6, -95.0), turned to 0 degrees
- moved J2 419.7 mm to (-199.0, -22.9), turned to 270 degrees
- moved R6 403.9 mm to (-78.9, -57.8)
- moved R7 401.4 mm to (-78.9, -52.9)
- moved R8 397.5 mm to (-133.0, -57.0), turned to 270 degrees
- moved D3 397.4 mm to (-137.8, -40.8)
- moved R9 394.4 mm to (-140.7, -56.7)
- moved J3 392.2 mm to (-53.6, -40.4)
- moved R10 391.6 mm to (-85.5, -30.2)
- moved R12 390.2 mm to (-64.0, -30.3)
- moved Q1 384.6 mm to (-122.6, -49.1), turned to 90 degrees
- moved C8 373.1 mm to (-79.0, -65.2), turned to 180 degrees
- moved R11 370.9 mm to (-80.2, -30.2), turned to 90 degrees
- moved C7 366.5 mm to (-78.9, -72.3), turned to 180 degrees
- moved D2 365.9 mm to (-90.7, -87.9), turned to 270 degrees
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Connections:
- J4 pad 2: GND -> Net-(C7-Pad1)
- R6 pad 1: GND -> Net-(C7-Pad1)
- RV1 pad 1: Net-(C7-Pad1) -> GND
- RV1 pad 3: GND -> Net-(C7-Pad1)
Routing:
- net GND: track 0.00 -> 861.4 mm
- net ADC_5V_0: track 0.00 -> 272.8 mm
- net v24: track 0.00 -> 268.7 mm
- net GND_ENB: track 0.00 -> 142.5 mm
- net ADC_ADJS_3: track 0.00 -> 121.9 mm
- net ADC_24S_5: track 0.00 -> 108.9 mm
- net Net-(C7-Pad1): track 0.00 -> 98.1 mm
- net ADC_ADJ_2: track 0.00 -> 96.8 mm
- net ADC_24V_4: track 0.00 -> 84.9 mm
- net PWR_ENABLE: track 0.00 -> 72.1 mm
- net LCD_DATA: track 0.00 -> 57.6 mm
- net Net-(RV1-Pad2): track 0.00 -> 56.9 mm
- net LCD_RE: track 0.00 -> 49.0 mm
- net LCD_CK: track 0.00 -> 46.4 mm
- net Net-(D2-Pad1): track 0.00 -> 39.4 mm
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Other:
- net class Default: clearance 0.4 -> 0.6; trace_width 0.5 -> 0.6; via_dia 0.8 -> 0.6
- net class pwr added: clearance 1, trace_width 1, via_dia 0.8, via_drill 0.4
- rule trace_clearance: 0.4 -> 0.6
